Commit message: Gazeboo Update

File: simulation/urdf/aerial_v1.urdf (robot description, URDF)
Before this commit: robot sentinel_aerial_v1, 21 links, 20 joints
Links:
- added link lidar_link, mass 0.025; collision cylinder length=0.020 radius=0.018; visual cylinder length=0.020 radius=0.018
Joints:
- added joint joint_lidar: type fixed, parent base_link, child lidar_link, origin xyz=0 0 0.035 rpy=0 0 0
- joint joint_prop_fr: axis 0 0 -1 -> 0 0 1
- joint joint_prop_rl: axis 0 0 -1 -> 0 0 1
